File: RaspberryPi-I2C-LevelShifter.sch (KiCad schematic (older format))
At the start: 15 parts, among them P1 CONN_13X2, P2 CONN_2, P3 CONN_2, P4 CONN_4_GROVE, U1 TCA9517A

Commit message: correct according last library changes
Parts:
- removed P1: CONN_13X2, symbol CONN_13X2
- removed P2, P3: CONN_2, symbol CONN_2
- added P?: CONN_02X13, symbol CONN_02X13
- added P? (x2): CONN_01X02, symbol CONN_01X02
Other:
- moved on the sheet: C1, C2, C3, C4
